File: MQTemp.kicad_pcb (KiCad board)
At the start: 2 copper layers, 42.5 x 38.1 mm, 10 parts, among them J1 Conn_01x02_Male, SW1 SW_DIP_x01

Commit message: Changed input voltage to 3.3V
Parts:
- R3: value 4k7 -> 3k3
Connections:
- WEMOSD1mini1 pad 8: unconnected-(WEMOSD1mini1-Pad8) -> VCC
- WEMOSD1mini1 pad 9: VCC -> unconnected-(WEMOSD1mini1-Pad9)
Routing:
- net VCC: track 51.4 -> 72.1 mm
Other:
- board text added: "3V3"
Changed lines of the file:
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@@
   (net 8 "unconnected-(WEMOSD1mini1-Pad6)")
   (net 9 "unconnected-(WEMOSD1mini1-Pad7)")
-  (net 10 "unconnected-(WEMOSD1mini1-Pad8)")
+  (net 10 "unconnected-(WEMOSD1mini1-Pad9)")
   (net 11 "unconnected-(WEMOSD1mini1-Pad11)")
   (net 12 "unconnected-(WEMOSD1mini1-Pad12)")
@@
       (effects (font (size 1 1) (thickness 0.15)))
     )
-    (fp_text value "4k7" (at 5.08 2.37 -90) (layer "F.Fab")
+    (fp_text value "3k3" (at 5.08 2.37 -90) (layer "F.Fab")
       (effects (font (size 1 1) (thickness 0.15)))
     )
@@
       (net 9 "unconnected-(WEMOSD1mini1-Pad7)") (pinfunction "CS/D8") (pintype "bidirectional+no_connect"))
     (pad "8" thru_hole oval (at 0 17.78) (size 2 1.6) (drill 1) (layers *.Cu *.Mask)
-      (net 10 "unconnected-(WEMOSD1mini1-Pad8)") (pinfunction "3V3") (pintype "power_out+no_connect"))
+      (net 2 "VCC") (pinfunction "3V3") (pintype "power_out"))
     (pad "9" thru_hole oval (at 22.86 17.78) (size 2 1.6) (drill 1) (layers *.Cu *.Mask)
-      (net 2 "VCC") (pinfunction "5V") (pintype "power_in"))
+      (net 10 "unconnected-(WEMOSD1mini1-Pad9)") (pinfunction "5V") (pintype "power_in+no_connect"))
     (pad "10" thru_hole oval (at 22.86 15.24) (size 2 1.6) (drill 1) (layers *.Cu *.Mask)
       (net 3 "GND") (pinfunction "GND") (pintype "power_in"))
@@
     (effects (font (size 1 1) (thickness 0.15)) (justify mirror))
   )
+  (gr_text "3V3" (at 57.785 64.77) (layer "B.SilkS")
+    (effects (font (size 1 1) (thickness 0.15)) (justify mirror))
+  )
   (gr_text "RST" (at 58.42 46.99) (layer "B.SilkS")
     (effects (font (size 1 1) (thickness 0.15)) (justify mirror))
@@
     (effects (font (size 1 1) (thickness 0.15)) (justify mirror))
   )
+  (gr_text "3V3" (at 57.785 64.77) (layer "F.SilkS")
+    (effects (font (size 1 1) (thickness 0.15)))
+  )
   (gr_text "RST" (at 57.785 45.72) (layer "F.SilkS")
     (effects (font (size 1 1) (thickness 0.15)))
@@
   (segment (start 63.5 49.53) (end 61.05 49.53) (width 0.25) (layer "F.Cu") (net 1))
   (segment (start 90.805 40.005) (end 87.63 40.005) (width 0.25) (layer "F.Cu") (net 2))
-  (segment (start 92.71 46.985) (end 92.71 68.58) (width 0.25) (layer "B.Cu") (net 2))
-  (segment (start 84.005 68.585) (end 92.705 68.585) (width 0.25) (layer "B.Cu") (net 2))
+  (segment (start 92.71 46.985) (end 92.71 60.96) (width 0.25) (layer "B.Cu") (net 2))
+  (segment (start 64.86 60.96) (end 61.05 64.77) (width 0.25) (layer "B.Cu") (net 2))
   (segment (start 92.71 68.58) (end 92.705 68.585) (width 0.25) (layer "B.Cu") (net 2))
   (segment (start 95.61 50.165) (end 95.61 49.89) (width 0.25) (layer "B.Cu") (net 2))
   (segment (start 95.61 49.89) (end 92.705 46.985) (width 0.25) (layer "B.Cu") (net 2))
-  (segment (start 83.91 68.49) (end 84.005 68.585) (width 0.25) (layer "B.Cu") (net 2))
   (segment (start 92.71 45.085) (end 90.805 43.18) (width 0.25) (layer "B.Cu") (net 2))
   (segment (start 92.705 68.585) (end 94.615 68.585) (width 0.25) (layer "B.Cu") (net 2))
-  (segment (start 83.91 64.77) (end 83.91 68.49) (width 0.25) (layer "B.Cu") (net 2))
   (segment (start 90.805 43.18) (end 90.805 40.005) (width 0.25) (layer "B.Cu") (net 2))
+  (segment (start 92.71 60.96) (end 92.71 68.58) (width 0.25) (layer "B.Cu") (net 2))
+  (segment (start 92.71 60.96) (end 64.86 60.96) (width 0.25) (layer "B.Cu") (net 2))
   (segment (start 92.705 45.085) (end 92.705 46.985) (width 0.25) (layer "B.Cu") (net 2))
   (segment (start 95.61 58.06) (end 95.61 52.705) (width 0.25) (layer "F.Cu") (net 3))
