File: MQTemp.kicad_pcb (KiCad board)
At the start: 2 copper layers, 42.5 x 38.1 mm, 10 parts, among them J1 Conn_01x02_Male, SW1 SW_DIP_x01

Commit message: Added filled zones
Connections:
- net Net-(R1-Pad2) renamed /BATT
Routing:
- net VCC: track 51.4 -> 3.45 mm
- net GND: track 45.3 -> 0.00 mm
- net /D6: track 63.7 -> 36.7 mm
- net /D5: track 36.1 -> 12.5 mm
- net /BATT: track 38.3 -> 21.3 mm
- added copper zone on F.Cu, net /BATT
- added copper zone on B.Cu, net /D5
- added copper zone on F.Cu, net /D6
- added copper zone on B.Cu, net GND
- added copper zone on F.Cu, net GND
- added copper zone on B.Cu, net VCC
- added copper zone on F.Cu, net VCC
